File: Hardware/RedFive.sch (EAGLE design)
At the start: 82 parts, among them IC3 LM1117, J1 AMP FCI 10103594-0001LF, J3 POWER_JACKSUPER_BOMB_DIGITY, J5 CORTEX_JTAG_DEBUG_SMD, Q1 1A/60V/500mΩ, U1 CH340C, U2 1.8V, U3 AP2112-3.3V, U4 FE310, U5 32MB, Y1 32.768KHZ, Y2 16MHz

Commit message: pre review changes
Parts:
- C16: device SparkFun-Capacitors:1.0UF-16V-10%(0603) -> SparkFun-Capacitors:1.0UF-0603-16V-10%
- C17: device SparkFun-Capacitors:10NF/10000PF-50V-10%(0603) -> SparkFun-Capacitors:10NF-0603-50V-10%
- JP11: device SparkFun-Connectors:M08SMD-COMBO -> SparkFun-Connectors:CONN_08SMD-COMBO-FEMALE
- JP13: device SparkFun-Connectors:M06SMD-STRAIGHT-COMBO -> SparkFun-Connectors:CONN_06SMD-STRAIGHT-COMBO-FEMALE
- JP2: value M10SMD_COMBO -> (none); device SparkFun-Connectors:M10SMD_COMBO -> SparkFun-Connectors:CONN_10SMD_COMBO-FEMALE
- Q1: value 1A/60V/500mΩ -> 1.1A/60V/600mΩ; device SparkFun-DiscreteSemi:MOSFET-PCH-ZXMP6A13F -> SparkFun-DiscreteSemi:MOSFET_PCH-SI2309DS
Other:
- moved on the sheet: JP11, JP13

Commit message: post review changes
Parts:
- removed J1: AMP FCI 10103594-0001LF, SparkFun-Connectors:USB_MICRO-B_HALF_PTH_MILL
- added J2: USB Female Type C Connector, SparkFun-Connectors:USB_C
- added R18, R19: 5.1k, SparkFun-Resistors:5.1KOHM5.1KOHM-0603-1/10W-1%
- added TP1, TP2, TP3, TP4, TP5: TEST-POINT3, SparkFun-Connectors:TEST-POINT3
- LED2: value GREEN -> RED; device SparkFun-LED:LED-GREEN_HIDDENSILK -> SparkFun-LED:LED-RED1206; PROD_ID DIO-09910 -> (none)
Connections:
- new net N$12: J2.CC2, R18.2
- new net N$17: J2.CC1, R19.2
- net !RESET: now also TP5.1
- net GND: now also J2.GND, J2.SHLD, R18.1, R19.1; no longer J1.GND, J1.SHIELD
- net N$13: now also J2.D-; no longer J1.D-
- net N$14: now also J2.D+; no longer J1.D+
- net TCK: now also TP2.1
- net TDI: now also TP4.1
- net TDO: now also TP3.1
- net TMS: now also TP1.1
- net VUSB: now also J2.VBUS; no longer J1.VBUS
Other:
- moved on the sheet: C10, C12, C15, C17, C18, D2, D3, D4, F1, LED5, R12, R16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

Commit message: design review checklist
Parts:
- J2: device SparkFun-Connectors:USB_C -> SparkFun-Connectors:USB_C2-LAYER
Changed lines of the file:
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@@
 <?xml version="1.0" encoding="utf-8"?>
 <!DOCTYPE eagle SYSTEM "eagle.dtd">
-<eagle version="9.3.1">
+<eagle version="9.1.0">
 <drawing>
 <settings>
@@
 <part name="GND27" library="SparkFun-PowerSymbols" deviceset="GND" device=""/>
 <part name="SUPPLY17" library="SparkFun-PowerSymbols" deviceset="VIN" device=""/>
-<part name="J2" library="SparkFun-Connectors" deviceset="USB_C" device="" value="USB Female Type C Connector"/>
+<part name="J2" library="SparkFun-Connectors" deviceset="USB_C" device="2-LAYER" value="USB Female Type C Connector"/>
 <part name="R18" library="SparkFun-Resistors" deviceset="5.1KOHM" device="5.1KOHM-0603-1/10W-1%" value="5.1k"/>
 <part name="R19" library="SparkFun-Resistors" deviceset="5.1KOHM" device="5.1KOHM-0603-1/10W-1%" value="5.1k"/>
@@
 </instance>
 <instance part="J2" gate="J1" x="12.7" y="25.4" smashed="yes">
-<attribute name="VALUE" x="10.16" y="12.954" size="1.778" layer="96" font="vector" rot="MR180" align="top-left"/>
 <attribute name="NAME" x="10.16" y="35.814" size="1.778" layer="95" font="vector"/>
 </instance>

Commit message: Adding prod_id to JTAG
Parts:
- J5: value CORTEX_JTAG_DEBUG_SMD -> JTAG
Changed lines of the file:
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@@
 <part name="GND17" library="SparkFun-PowerSymbols" deviceset="GND" device=""/>
 <part name="U4" library="SparkFun-IC-Microcontroller" deviceset="SIFIVE_FE310" device="" value="FE310"/>
-<part name="J5" library="SparkFun-Connectors" deviceset="CORTEX_JTAG_DEBUG" device="_SMD"/>
+<part name="J5" library="SparkFun-Connectors" deviceset="CORTEX_JTAG_DEBUG" device="_SMD" value="JTAG"/>
 <part name="GND1" library="SparkFun-PowerSymbols" deviceset="GND" device=""/>
 <part name="SUPPLY10" library="SparkFun-PowerSymbols" deviceset="3.3V" device=""/>

Commit message: v02
Parts:
- removed D3: YELLOW, SparkFun-LED:LED-YELLOW_HIDDENSILK
- removed LED5: GREEN, SparkFun-LED:LED-GREENLILYPAD
- removed R11, R13, R17: 22, SparkFun-Resistors:22OHM-0603-1/10W-1%
- removed R12, R16: 4.7k, SparkFun-Resistors:4.7KOHM-0603-1/10W-1%
- removed U1: CH340C, SparkFun-IC-Comms:CH340C
- added C27, C28, C29: 0.1uF, SparkFun-Capacitors:0.1UF-0603-25V-(+80/-20%)
- added C30: 10uF, SparkFun-Capacitors:10UF-0603-6.3V-20%
- added D5: YELLOW, SparkFun-LED:LED-YELLOW_HIDDENSILK
- added J1: AVR_SPI_PROG_3X2PTH, SparkFun-Connectors:AVR_SPI_PROG_3X2PTH
- added LED3: GREEN, SparkFun-LED:LED-GREENLILYPAD
- added R20: 100k, SparkFun-Resistors:100KOHM-0603-1/10W-1%
- added R21, R22: 4.7k, SparkFun-Resistors:4.7KOHM-0603-1/10W-1%
- added TP6, TP7, TP8: TEST-POINT3, SparkFun-Connectors:TEST-POINT3
- added U$44: MK22FN128VLH10, SparkFun-IC-Comms:MK22FN128VLH10
- C17: value 10nF -> 0.1uF; device SparkFun-Capacitors:10NF-0603-50V-10% -> SparkFun-Capacitors:0.1UF-0603-25V-(+80/-20%)
Connections:
- removed net N$11: JP2.7, R11.2
- removed net N$14: J2.D+, U1.UD+
- removed net N$16: JP2.5, R17.2
- removed net N$4: JP2.6, R13.2
- removed net N$5: LED5.A, R16.1
- removed net N$9: D3.A, R12.1
- new net D+: J2.D+, U$44.D+
- new net D-: J2.D-, U$44.D-
- new net DBG_RESET: J1.4, R20.1, TP8.1, U$44.RESET_B
- new net DBG_SWDCLK: J1.3, U$44.PTA0
- new net DBG_SWDIO: J1.1, U$44.PTA3
- new net DBG_SWO: J1.5, U$44.PTA2
- net !RESET: now also U$44.PTD7; no longer U1.!DTR
- net 3.3V: now also C17.1, C18.1, C27.1, C28.1, C29.1, C30.1, J1.2, R20.2, R21.2, R22.2, TP6.1, U$44.PTA4/LLWU_P3, U$44.USBVDD, U$44.VBATT, U$44.VDD, U$44.VDDA, U$44.VREFH
- net 5V: no longer C18.1, R12.2, R16.2, U1.VCC
- net GND: now also C27.2, C28.2, C29.2, C30.2, J1.6, TP7.1, U$44.GND, U$44.VREFL, U$44.VSSA; no longer U1.GND
- net N$13: now also D5.A, R21.1; no longer J2.D-, U1.UD-
- net N$6: now also LED3.A, R22.1; no longer C17.1, U1.V3
- net RXI: now also D5.C, U$44.PTB16; no longer D3.C, U1.TXO
- net SPI_MISO: now also JP2.6; no longer R13.1
- net SPI_MOSI: now also JP2.7; no longer R11.1
- net SPI_SCK: now also JP2.5; no longer R17.1
- net TCK: now also U$44.PTD5
- net TDI: now also U$44.PTD2/LLWU_P13
- net TDO: now also U$44.PTE1/LLWU_P0
- net TMS: now also U$44.PTD6/LLWU_P15
- net TXO: now also LED3.C, U$44.PTB17; no longer LED5.C, U1.RXI
Other:
- note added: "Programming Headers"
- note removed: "JTAG Header"
- moved on the sheet: C11, C13, C14, C19, C2, C20, C21, C22, C6, C7, C8, J4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

Commit message: pre design review number 2
Other:
- note added: "USB -> JTAG"
- note added: "v02"
- moved on the sheet: C2, R5, U5
Changed lines of the file:
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@@
 <wire x1="137.16" y1="48.26" x2="137.16" y2="93.98" width="0.1524" layer="97" style="longdash"/>
 <wire x1="137.16" y1="93.98" x2="137.16" y2="129.54" width="0.1524" layer="97" style="longdash"/>
-<wire x1="137.16" y1="129.54" x2="137.16" y2="185.42" width="0.1524" layer="97" style="longdash"/>
+<wire x1="137.16" y1="129.54" x2="137.16" y2="147.32" width="0.1524" layer="97" style="longdash"/>
+<wire x1="137.16" y1="147.32" x2="137.16" y2="185.42" width="0.1524" layer="97" style="longdash"/>
 <wire x1="137.16" y1="129.54" x2="0" y2="129.54" width="0.1524" layer="97" style="longdash"/>
 <text x="86.36" y="88.9" size="2.54" layer="94" font="vector">Qwiic</text>
@@
 <text x="2.54" y="124.46" size="2.54" layer="94" font="vector">Capacitors</text>
 <text x="166.116" y="11.43" size="2.54" layer="94" font="vector">Andrew England</text>
-<text x="236.22" y="7.874" size="2.54" layer="94" font="vector">v01</text>
+<text x="236.22" y="7.874" size="2.54" layer="94" font="vector">v02</text>
 <wire x1="137.16" y1="48.26" x2="137.16" y2="40.64" width="0.1524" layer="97" style="longdash"/>
 <wire x1="137.16" y1="40.64" x2="147.32" y2="40.64" width="0.1524" layer="97" style="longdash"/>
@@
 <wire x1="137.16" y1="93.98" x2="83.82" y2="93.98" width="0.1524" layer="97" style="longdash"/>
 <wire x1="83.82" y1="93.98" x2="83.82" y2="48.26" width="0.1524" layer="97" style="longdash"/>
+<wire x1="248.92" y1="147.32" x2="137.16" y2="147.32" width="0.1524" layer="97" style="longdash"/>
+<text x="139.954" y="143.002" size="2.54" layer="94" font="vector">USB -&gt; JTAG</text>
 </plain>
 <instances>
@@
 <attribute name="VALUE" x="119.38" y="53.086" size="1.778" layer="96" align="top-center"/>
 </instance>
-<instance part="U5" gate="G$1" x="182.88" y="154.94" smashed="yes">
-<attribute name="NAME" x="172.72" y="144.78" size="1.778" layer="95" font="vector"/>
-<attribute name="VALUE" x="172.72" y="165.608" size="1.778" layer="96" font="vector"/>
-</instance>
-<instance part="C2" gate="G$1" x="167.64" y="154.94" smashed="yes" rot="MR0">
-<attribute name="NAME" x="166.116" y="157.861" size="1.778" layer="95" font="vector" rot="MR0"/>
-<attribute name="VALUE" x="166.116" y="152.781" size="1.778" layer="96" font="vector" rot="MR0"/>
-</instance>
-<instance part="GND5" gate="1" x="167.64" y="144.78" smashed="yes">
-<attribute name="VALUE" x="167.64" y="144.526" size="1.778" layer="96" align="top-center"/>
-</instance>
-<instance part="SUPPLY14" gate="G$1" x="167.64" y="165.1" smashed="yes">
-<attribute name="VALUE" x="167.64" y="167.894" size="1.778" layer="96" align="bottom-center"/>
-</instance>
-<instance part="R5" gate="G$1" x="213.36" y="160.02" smashed="yes" rot="R90">
-<attribute name="NAME" x="211.836" y="160.02" size="1.778" layer="95" font="vector" rot="R90" align="bottom-center"/>
-<attribute name="VALUE" x="214.884" y="160.02" size="1.778" layer="96" font="vector" rot="R90" align="top-center"/>
-</instance>
-<instance part="SUPPLY15" gate="G$1" x="213.36" y="167.64" smashed="yes">
-<attribute name="VALUE" x="213.36" y="170.434" size="1.778" layer="96" align="bottom-center"/>
+<instance part="U5" gate="G$1" x="182.88" y="162.56" smashed="yes">
+<attribute name="NAME" x="172.72" y="152.4" size="1.778" layer="95" font="vector"/>
+<attribute name="VALUE" x="172.72" y="173.228" size="1.778" layer="96" font="vector"/>
+</instance>
+<instance part="C2" gate="G$1" x="167.64" y="162.56" smashed="yes" rot="MR0">
+<attribute name="NAME" x="166.116" y="165.481" size="1.778" layer="95" font="vector" rot="MR0"/>
+<attribute name="VALUE" x="166.116" y="160.401" size="1.778" layer="96" font="vector" rot="MR0"/>
+</instance>
+<instance part="GND5" gate="1" x="167.64" y="152.4" smashed="yes">
+<attribute name="VALUE" x="167.64" y="152.146" size="1.778" layer="96" align="top-center"/>
+</instance>
+<instance part="SUPPLY14" gate="G$1" x="167.64" y="172.72" smashed="yes">
+<attribute name="VALUE" x="167.64" y="175.514" size="1.778" layer="96" align="bottom-center"/>
+</instance>
+<instance part="R5" gate="G$1" x="213.36" y="167.64" smashed="yes" rot="R90">
+<attribute name="NAME" x="211.836" y="167.64" size="1.778" layer="95" font="vector" rot="R90" align="bottom-center"/>
+<attribute name="VALUE" x="214.884" y="167.64" size="1.778" layer="96" font="vector" rot="R90" align="top-center"/>
+</instance>
+<instance part="SUPPLY15" gate="G$1" x="213.36" y="175.26" smashed="yes">
+<attribute name="VALUE" x="213.36" y="178.054" size="1.778" layer="96" align="bottom-center"/>
 </instance>
 <instance part="C6" gate="G$1" x="15.24" y="106.68" smashed="yes">
@@
 <pinref part="C2" gate="G$1" pin="2"/>
 <pinref part="U5" gate="G$1" pin="GND"/>
-<wire x1="167.64" y1="152.4" x2="167.64" y2="149.86" width="0.1524" layer="91"/>
-<wire x1="167.64" y1="149.86" x2="170.18" y2="149.86" width="0.1524" layer="91"/>
-<wire x1="167.64" y1="149.86" x2="167.64" y2="147.32" width="0.1524" layer="91"/>
-<junction x="167.64" y="149.86"/>
+<wire x1="167.64" y1="160.02" x2="167.64" y2="157.48" width="0.1524" layer="91"/>
+<wire x1="167.64" y1="157.48" x2="170.18" y2="157.48" width="0.1524" layer="91"/>
+<wire x1="167.64" y1="157.48" x2="167.64" y2="154.94" width="0.1524" layer="91"/>
+<junction x="167.64" y="157.48"/>
 <pinref part="GND5" gate="1" pin="GND"/>
 </segment>
@@
 <segment>
 <pinref part="U5" gate="G$1" pin="VCC"/>
-<wire x1="170.18" y1="162.56" x2="167.64" y2="162.56" width="0.1524" layer="91"/>
+<wire x1="170.18" y1="170.18" x2="167.64" y2="170.18" width="0.1524" layer="91"/>
 <pinref part="C2" gate="G$1" pin="1"/>
-<wire x1="167.64" y1="162.56" x2="167.64" y2="160.02" width="0.1524" layer="91"/>
-<wire x1="167.64" y1="162.56" x2="167.64" y2="165.1" width="0.1524" layer="91"/>
-<junction x="167.64" y="162.56"/>
+<wire x1="167.64" y1="170.18" x2="167.64" y2="167.64" width="0.1524" layer="91"/>
+<wire x1="167.64" y1="170.18" x2="167.64" y2="172.72" width="0.1524" layer="91"/>
+<junction x="167.64" y="170.18"/>
 <pinref part="SUPPLY14" gate="G$1" pin="3.3V"/>
 </segment>
 <segment>
 <pinref part="R5" gate="G$1" pin="2"/>
-<wire x1="213.36" y1="165.1" x2="213.36" y2="167.64" width="0.1524" layer="91"/>
+<wire x1="213.36" y1="172.72" x2="213.36" y2="175.26" width="0.1524" layer="91"/>
 <pinref part="SUPPLY15" gate="G$1" pin="3.3V"/>
 </segment>
@@
 <net name="QSPI_3" class="0">
 <segment>
-<wire x1="195.58" y1="152.4" x2="213.36" y2="152.4" width="0.1524" layer="91"/>
+<wire x1="195.58" y1="160.02" x2="213.36" y2="160.02" width="0.1524" layer="91"/>
 <pinref part="U5" gate="G$1" pin="HOLD#/IO3"/>
-<label x="215.9" y="152.4" size="1.27" layer="95" font="vector" xref="yes"/>
+<label x="215.9" y="160.02" size="1.27" layer="95" font="vector" xref="yes"/>
 <pinref part="R5" gate="G$1" pin="1"/>
-<wire x1="213.36" y1="152.4" x2="215.9" y2="152.4" width="0.1524" layer="91"/>
-<wire x1="213.36" y1="154.94" x2="213.36" y2="152.4" width="0.1524" layer="91"/>
-<junction x="213.36" y="152.4"/>
+<wire x1="213.36" y1="160.02" x2="215.9" y2="160.02" width="0.1524" layer="91"/>
+<wire x1="213.36" y1="162.56" x2="213.36" y2="160.02" width="0.1524" layer="91"/>
+<junction x="213.36" y="160.02"/>
 </segment>
 </net>
 <net name="QSPI_2" class="0">
 <segment>
-<wire x1="195.58" y1="154.94" x2="198.12" y2="154.94" width="0.1524" layer="91"/>
+<wire x1="195.58" y1="162.56" x2="198.12" y2="162.56" width="0.1524" layer="91"/>
 <pinref part="U5" gate="G$1" pin="WP#/IO2"/>
-<label x="198.12" y="154.94" size="1.27" layer="95" font="vector" xref="yes"/>
+<label x="198.12" y="162.56" size="1.27" layer="95" font="vector" xref="yes"/>
 </segment>
 </net>
 <net name="QSPI_0" class="0">
 <segment>
-<wire x1="195.58" y1="160.02" x2="198.12" y2="160.02" width="0.1524" layer="91"/>
+<wire x1="195.58" y1="167.64" x2="198.12" y2="167.64" width="0.1524" layer="91"/>
 <pinref part="U5" gate="G$1" pin="MOSI/IO0"/>
-<label x="198.12" y="160.02" size="1.27" layer="95" font="vector" xref="yes"/>
+<label x="198.12" y="167.64" size="1.27" layer="95" font="vector" xref="yes"/>
 </segment>
 </net>
 <net name="QSPI_SCK" class="0">
 <segment>
-<wire x1="195.58" y1="162.56" x2="198.12" y2="162.56" width="0.1524" layer="91"/>
+<wire x1="195.58" y1="170.18" x2="198.12" y2="170.18" width="0.1524" layer="91"/>
 <pinref part="U5" gate="G$1" pin="SCK"/>
-<label x="198.12" y="162.56" size="1.27" layer="95" font="vector" xref="yes"/>
+<label x="198.12" y="170.18" size="1.27" layer="95" font="vector" xref="yes"/>
 </segment>
 </net>
 <net name="QSPI_1" class="0">
 <segment>
+<wire x1="195.58" y1="165.1" x2="198.12" y2="165.1" width="0.1524" layer="91"/>
+<pinref part="U5" gate="G$1" pin="MISO/IO1"/>
+<label x="198.12" y="165.1" size="1.27" layer="95" font="vector" xref="yes"/>
+</segment>
+</net>
+<net name="QSPI_CS" class="0">
+<segment>
 <wire x1="195.58" y1="157.48" x2="198.12" y2="157.48" width="0.1524" layer="91"/>
-<pinref part="U5" gate="G$1" pin="MISO/IO1"/>
+<pinref part="U5" gate="G$1" pin="CE#"/>
 <label x="198.12" y="157.48" size="1.27" layer="95" font="vector" xref="yes"/>
 </segment>
 </net>
-<net name="QSPI_CS" class="0">
-<segment>
-<wire x1="195.58" y1="149.86" x2="198.12" y2="149.86" width="0.1524" layer="91"/>
-<pinref part="U5" gate="G$1" pin="CE#"/>
-<label x="198.12" y="149.86" size="1.27" layer="95" font="vector" xref="yes"/>
-</segment>
-</net>
