File: Hardware/RedFive.sch (EAGLE design)
At the start: 96 parts, among them IC3 LM1117, J1 FEMALE 2x3, J2 USB Female Type C Connector, J3 POWER_JACKSUPER_BOMB_DIGITY, J4 QWIIC_RIGHT_ANGLE, J5 JTAG, Q1 1.1A/60V/600mΩ, U2 1.8V, U3 AP2112-3.3V, U4 FE310, U5 32MBit, Y1 32.768KHZ, Y2 16MHz

Commit message: Pre design review-reds
Parts:
- removed TP1, TP2, TP3, TP4, TP5, TP6, TP7: TEST-POINT3, SparkFun-Connectors:TEST-POINT3
- J1: device SparkFun-Connectors:CONN_03X2FEMALE -> SparkFun-Connectors:CONN_03X2POGO_PINS
- J5: value JTAG -> CORTEX_JTAG_DEBUG_PTH_NS; device SparkFun-Connectors:CORTEX_JTAG_DEBUG_SMD -> SparkFun-Connectors:CORTEX_JTAG_DEBUG_PTH_NS
Connections:
- net !RESET: no longer TP5.1
- net 3.3V: no longer TP6.1
- net GND: no longer TP7.1
- net TCK: no longer TP2.1
- net TDI: no longer TP4.1
- net TDO: no longer TP3.1
- net TMS: no longer TP1.1
Changed lines of the file:
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@@
 <?xml version="1.0" encoding="utf-8"?>
 <!DOCTYPE eagle SYSTEM "eagle.dtd">
-<eagle version="9.1.0">
+<eagle version="9.3.1">
 <drawing>
 <settings>
@@
 <part name="GND17" library="SparkFun-PowerSymbols" deviceset="GND" device=""/>
 <part name="U4" library="SparkFun-IC-Microcontroller" deviceset="SIFIVE_FE310" device="" value="FE310"/>
-<part name="J5" library="SparkFun-Connectors" deviceset="CORTEX_JTAG_DEBUG" device="_SMD" value="JTAG"/>
+<part name="J5" library="SparkFun-Connectors" deviceset="CORTEX_JTAG_DEBUG" device="_PTH_NS" value="CORTEX_JTAG_DEBUG_PTH_NS"/>
 <part name="GND1" library="SparkFun-PowerSymbols" deviceset="GND" device=""/>
 <part name="SUPPLY10" library="SparkFun-PowerSymbols" deviceset="3.3V" device=""/>
@@
 <part name="GND29" library="SparkFun-PowerSymbols" deviceset="GND" device=""/>
 <part name="GND31" library="SparkFun-PowerSymbols" deviceset="GND" device=""/>
-<part name="TP1" library="SparkFun-Connectors" deviceset="TEST-POINT" device="3"/>
-<part name="TP2" library="SparkFun-Connectors" deviceset="TEST-POINT" device="3"/>
-<part name="TP3" library="SparkFun-Connectors" deviceset="TEST-POINT" device="3"/>
-<part name="TP4" library="SparkFun-Connectors" deviceset="TEST-POINT" device="3"/>
-<part name="TP5" library="SparkFun-Connectors" deviceset="TEST-POINT" device="3"/>
-<part name="TP6" library="SparkFun-Connectors" deviceset="TEST-POINT" device="3"/>
-<part name="TP7" library="SparkFun-Connectors" deviceset="TEST-POINT" device="3"/>
 <part name="U$44" library="SparkFun-IC-Comms" deviceset="MK22FN128VLH10" device="" value="MK22FN128VLH10"/>
 <part name="SUPPLY7" library="SparkFun-PowerSymbols" deviceset="3.3V" device=""/>
 <part name="C27" library="SparkFun-Capacitors" deviceset="0.1UF" device="-0603-25V-(+80/-20%)" value="0.1uF"/>
 <part name="GND32" library="SparkFun-PowerSymbols" deviceset="GND" device=""/>
-<part name="J1" library="SparkFun-Connectors" deviceset="CONN_03X2" device="FEMALE" value="FEMALE 2x3"/>
+<part name="J1" library="SparkFun-Connectors" deviceset="CONN_03X2" device="POGO_PINS" value="FEMALE 2x3"/>
 <part name="SUPPLY18" library="SparkFun-PowerSymbols" deviceset="3.3V" device=""/>
 <part name="GND24" library="SparkFun-PowerSymbols" deviceset="GND" device=""/>
@@
 <attribute name="VALUE" x="63.5" y="17.526" size="1.778" layer="96" align="top-center"/>
 </instance>
-<instance part="JP1" gate="G$1" x="76.2" y="55.88"/>
+<instance part="JP1" gate="G$1" x="76.2" y="55.88" smashed="yes">
+<attribute name="NAME" x="73.66" y="58.42" size="1.778" layer="95" font="vector"/>
+<attribute name="VALUE" x="73.66" y="53.34" size="1.778" layer="96" font="vector" align="top-left"/>
+</instance>
 </instances>
 <busses>
@@
 <instance part="J5" gate="J1" x="30.48" y="157.48" smashed="yes">
 <attribute name="NAME" x="17.78" y="165.354" size="1.778" layer="95" font="vector"/>
-<attribute name="VALUE" x="17.78" y="147.574" size="1.778" layer="96" font="vector"/>
 </instance>
 <instance part="GND1" gate="1" x="12.7" y="147.32" smashed="yes">
@@
 <attribute name="VALUE" x="105.664" y="73.66" size="1.778" layer="96" font="vector" rot="R90" align="top-center"/>
 </instance>
-<instance part="TP1" gate="G$1" x="48.26" y="165.1" smashed="yes" rot="R90">
-<attribute name="NAME" x="48.26" y="162.56" size="1.778" layer="95" font="vector" rot="R90"/>
-</instance>
-<instance part="TP2" gate="G$1" x="50.8" y="165.1" smashed="yes" rot="R90">
-<attribute name="NAME" x="50.8" y="162.56" size="1.778" layer="95" font="vector" rot="R90"/>
-</instance>
-<instance part="TP3" gate="G$1" x="53.34" y="165.1" smashed="yes" rot="R90">
-<attribute name="NAME" x="53.34" y="162.56" size="1.778" layer="95" font="vector" rot="R90"/>
-</instance>
-<instance part="TP4" gate="G$1" x="55.88" y="165.1" smashed="yes" rot="R90">
-<attribute name="NAME" x="55.88" y="162.56" size="1.778" layer="95" font="vector" rot="R90"/>
-</instance>
-<instance part="TP5" gate="G$1" x="58.42" y="165.1" smashed="yes" rot="R90">
-<attribute name="NAME" x="58.42" y="162.56" size="1.778" layer="95" font="vector" rot="R90"/>
-</instance>
-<instance part="TP6" gate="G$1" x="10.16" y="162.56" smashed="yes" rot="R180">
-<attribute name="NAME" x="12.7" y="162.56" size="1.778" layer="95" font="vector" rot="R180"/>
-</instance>
-<instance part="TP7" gate="G$1" x="10.16" y="154.94" smashed="yes" rot="R180">
-<attribute name="NAME" x="12.7" y="154.94" size="1.778" layer="95" font="vector" rot="R180"/>
-</instance>
-<instance part="U$44" gate="G$1" x="193.04" y="83.82"/>
+<instance part="U$44" gate="G$1" x="193.04" y="83.82" smashed="yes">
+<attribute name="NAME" x="167.64" y="40.64" size="1.778" layer="95" font="vector"/>
+<attribute name="VALUE" x="167.64" y="132.08" size="1.778" layer="96" font="vector"/>
+</instance>
 <instance part="SUPPLY7" gate="G$1" x="162.56" y="134.62" smashed="yes">
 <attribute name="VALUE" x="162.56" y="137.414" size="1.778" layer="96" align="bottom-center"/>
@@
 <attribute name="VALUE" x="149.86" y="103.886" size="1.778" layer="96" align="top-center"/>
 </instance>
-<instance part="J1" gate="G$1" x="104.14" y="157.48" rot="MR0"/>
+<instance part="J1" gate="G$1" x="104.14" y="157.48" smashed="yes" rot="MR0">
+<attribute name="NAME" x="107.696" y="163.068" size="1.778" layer="95" font="vector" rot="MR0"/>
+</instance>
 <instance part="SUPPLY18" gate="G$1" x="91.44" y="162.56" smashed="yes">
 <attribute name="VALUE" x="91.44" y="165.354" size="1.778" layer="96" align="bottom-center"/>
@@
 <wire x1="15.24" y1="160.02" x2="12.7" y2="160.02" width="0.1524" layer="91"/>
 <wire x1="12.7" y1="160.02" x2="12.7" y2="157.48" width="0.1524" layer="91"/>
-<wire x1="12.7" y1="157.48" x2="12.7" y2="154.94" width="0.1524" layer="91"/>
-<wire x1="12.7" y1="154.94" x2="12.7" y2="152.4" width="0.1524" layer="91"/>
+<wire x1="12.7" y1="157.48" x2="12.7" y2="152.4" width="0.1524" layer="91"/>
 <wire x1="12.7" y1="152.4" x2="12.7" y2="149.86" width="0.1524" layer="91"/>
 <pinref part="J5" gate="J1" pin="GNDDTCT"/>
@@
 <junction x="12.7" y="157.48"/>
 <pinref part="GND1" gate="1" pin="GND"/>
-<pinref part="TP7" gate="G$1" pin="1"/>
-<wire x1="12.7" y1="154.94" x2="10.16" y2="154.94" width="0.1524" layer="91"/>
-<junction x="12.7" y="154.94"/>
 </segment>
 <segment>
@@
 <wire x1="12.7" y1="162.56" x2="12.7" y2="165.1" width="0.1524" layer="91"/>
 <pinref part="SUPPLY10" gate="G$1" pin="3.3V"/>
-<pinref part="TP6" gate="G$1" pin="1"/>
-<wire x1="12.7" y1="162.56" x2="10.16" y2="162.56" width="0.1524" layer="91"/>
-<junction x="12.7" y="162.56"/>
 </segment>
 <segment>
@@
 <segment>
 <pinref part="J5" gate="J1" pin="NC/TDI"/>
-<wire x1="45.72" y1="154.94" x2="55.88" y2="154.94" width="0.1524" layer="91"/>
+<wire x1="45.72" y1="154.94" x2="60.96" y2="154.94" width="0.1524" layer="91"/>
 <label x="60.96" y="154.94" size="1.27" layer="95" font="vector" xref="yes"/>
-<pinref part="TP4" gate="G$1" pin="1"/>
-<wire x1="55.88" y1="154.94" x2="60.96" y2="154.94" width="0.1524" layer="91"/>
-<wire x1="55.88" y1="165.1" x2="55.88" y2="154.94" width="0.1524" layer="91"/>
-<junction x="55.88" y="154.94"/>
 </segment>
 <segment>
@@
 <segment>
 <pinref part="J5" gate="J1" pin="SWDIO/TMS"/>
-<wire x1="45.72" y1="162.56" x2="48.26" y2="162.56" width="0.1524" layer="91"/>
 <label x="60.96" y="162.56" size="1.27" layer="95" font="vector" xref="yes"/>
-<pinref part="TP1" gate="G$1" pin="1"/>
-<wire x1="48.26" y1="162.56" x2="60.96" y2="162.56" width="0.1524" layer="91"/>
-<wire x1="48.26" y1="165.1" x2="48.26" y2="162.56" width="0.1524" layer="91"/>
-<junction x="48.26" y="162.56"/>
+<wire x1="45.72" y1="162.56" x2="60.96" y2="162.56" width="0.1524" layer="91"/>
 </segment>
 <segment>
@@
 <segment>
 <pinref part="J5" gate="J1" pin="SWO/TDO"/>
-<wire x1="45.72" y1="157.48" x2="53.34" y2="157.48" width="0.1524" layer="91"/>
 <label x="60.96" y="157.48" size="1.27" layer="95" font="vector" xref="yes"/>
-<pinref part="TP3" gate="G$1" pin="1"/>
-<wire x1="53.34" y1="157.48" x2="60.96" y2="157.48" width="0.1524" layer="91"/>
-<wire x1="53.34" y1="165.1" x2="53.34" y2="157.48" width="0.1524" layer="91"/>
-<junction x="53.34" y="157.48"/>
+<wire x1="45.72" y1="157.48" x2="60.96" y2="157.48" width="0.1524" layer="91"/>
 </segment>
 <segment>
@@
 <segment>
 <pinref part="J5" gate="J1" pin="SWDCLK/TCK"/>
-<wire x1="45.72" y1="160.02" x2="50.8" y2="160.02" width="0.1524" layer="91"/>
 <label x="60.96" y="160.02" size="1.27" layer="95" font="vector" xref="yes"/>
-<pinref part="TP2" gate="G$1" pin="1"/>
-<wire x1="50.8" y1="160.02" x2="60.96" y2="160.02" width="0.1524" layer="91"/>
-<wire x1="50.8" y1="165.1" x2="50.8" y2="160.02" width="0.1524" layer="91"/>
-<junction x="50.8" y="160.02"/>
+<wire x1="45.72" y1="160.02" x2="60.96" y2="160.02" width="0.1524" layer="91"/>
 </segment>
 <segment>
@@
 <segment>
 <pinref part="J5" gate="J1" pin="!RESET"/>
-<wire x1="45.72" y1="152.4" x2="58.42" y2="152.4" width="0.1524" layer="91"/>
+<wire x1="45.72" y1="152.4" x2="60.96" y2="152.4" width="0.1524" layer="91"/>
 <label x="60.96" y="152.4" size="1.27" layer="95" font="vector" xref="yes"/>
-<pinref part="TP5" gate="G$1" pin="1"/>
-<wire x1="58.42" y1="152.4" x2="60.96" y2="152.4" width="0.1524" layer="91"/>
-<wire x1="58.42" y1="165.1" x2="58.42" y2="152.4" width="0.1524" layer="91"/>
-<junction x="58.42" y="152.4"/>
-</segment>
-<segment>
+</segment>
+<segment>
