File: Hardware/RedFive.brd (EAGLE design)
At the start: 68.6 x 53.3 mm, 124 parts, among them IC3 LM1117, J1 AMP FCI 10103594-0001LF, J3 POWER_JACKSUPER_BOMB_DIGITY, J5 CORTEX_JTAG_DEBUG_SMD, Q1 1A/60V/500mΩ, U1 CH340C, U2 1.8V, U3 AP2112-3.3V, U4 FE310, U5 32MB, Y1 32.768KHZ, Y2 16MHz

Commit message: pre review changes
Parts:
- C16, C17: device SparkFun-Capacitors:0603-CAP -> SparkFun-Capacitors:0603
- JP11: device SparkFun-Connectors:1X08_SMD_COMBINED@1 -> SparkFun-Connectors:1X08_SMD_COMBINED
- JP2: value M10SMD_COMBO -> (none)
- Q1: value 1A/60V/500mΩ -> 1.1A/60V/600mΩ
- moved FRAME1 86.3 mm to (1.00, -17.0)
- moved U$16 3.00 mm to (2.54, 48.3)
- moved FRAME2 0.24 mm to (1.00, -17.0)
Connections:
- net IO10: now also JP13.3; no longer JP13.3A, JP13.3B
- net IO11: now also JP13.4; no longer JP13.4A, JP13.4B
- net IO18: now also JP11.3, JP11.3@2; no longer JP11.3A, JP11.3B
- net IO19: now also JP11.4, JP11.4@2; no longer JP11.4A, JP11.4B
- net IO20: now also JP11.5, JP11.5@2; no longer JP11.5A, JP11.5B
- net IO21: now also JP11.6, JP11.6@2; no longer JP11.6A, JP11.6B
- net IO22: now also JP11.7, JP11.7@2; no longer JP11.7A, JP11.7B
- net IO23: now also JP11.8, JP11.8@2; no longer JP11.8A, JP11.8B
- net IO9: now also JP13.2; no longer JP13.2A, JP13.2B
- net RXI: now also JP11.1, JP11.1@2; no longer JP11.1A, JP11.1B
- net SCL: now also JP13.6; no longer JP13.6A, JP13.6B
- net SDA: now also JP13.5; no longer JP13.5A, JP13.5B
- net TXO: now also JP11.2, JP11.2@2; no longer JP11.2A, JP11.2B
Other:
- board text added: "A. England"
- board text removed: "J. Lindblom, N. Seidle"

Commit message: post review changes
Parts:
- removed J1: AMP FCI 10103594-0001LF, SparkFun-Connectors:USB-MICROB-PTH-MILL
- added J2: USB Female Type C Connector, SparkFun-Connectors:USB-C-16P
- added R18, R19: 5.1k, SparkFun-Resistors:0603
- added TP1, TP2, TP3, TP4, TP5: TEST-POINT3, SparkFun-Connectors:PAD.03X.03
- LED2: value GREEN -> RED; device SparkFun-LED:LED-1206-HIDDENSILK -> SparkFun-LED:LED-1206
Connections:
- new net N$12: J2.B5, R18.2
- new net N$17: J2.A5, R19.2
- net !RESET: now also TP5.P$1
- net GND: now also J2.GND, J2.GND2, J2.SHLD1, J2.SHLD2, J2.SHLD3, J2.SHLD4, J2.SHLD5, J2.SHLD6, J2.SHLD7, J2.SHLD8, R18.1, R19.1; no longer J1.GND, J1.SHIELD, J1.SHIELD10, J1.SHIELD2, J1.SHIELD3, J1.SHIELD4, J1.SHIELD5, J1.SHIELD6, J1.SHIELD7, J1.SHIELD8, J1.SHIELD9
- net N$13: now also J2.A7, J2.B7; no longer J1.D-
- net N$14: now also J2.A6, J2.B6; no longer J1.D+
- net TCK: now also TP2.P$1
- net TDI: now also TP4.P$1
- net TDO: now also TP3.P$1
- net TMS: now also TP1.P$1
- net VUSB: now also J2.VBUS1, J2.VBUS2; no longer J1.VBUS
Routing:
- net GND: track 30.7 -> 15.3 mm
- net TDI: track 12.3 -> 17.6 mm, vias 0 -> 1
- net VUSB: track 21.1 -> 18.2 mm
- net TCK: track 16.7 -> 19.4 mm, vias 2 -> 3
- net N$14: track 11.0 -> 9.36 mm
- net N$13: track 11.0 -> 9.47 mm
- net !RESET: track 103.2 -> 104.0 mm, vias 5 -> 6
- net TMS: track 16.1 -> 16.0 mm, vias 2 -> 3

Commit message: design review checklist
Parts:
- moved R18 3.81 mm to (6.35, 33.0), turned to 180 degrees
- moved R19 3.81 mm to (2.54, 33.0), turned to 0 degrees
Routing:
- net N$17: track 0.00 -> 9.63 mm
- net GND: track 15.3 -> 24.8 mm, vias 63 -> 64
- net N$12: track 0.00 -> 7.72 mm
- net N$13: track 9.47 -> 11.9 mm
- net VUSB: track 18.2 -> 20.5 mm
- net N$14: track 9.36 -> 11.3 mm

Commit message: ordered prototypes
Parts:
- removed U$44: (no value), Redfive_logo#05#png (1):REDFIVE_LOGO#05#PNG
- added U$52: (no value), Redfive_logo#05#png (2):REDFIVE_LOGO#05#PNG
Changed lines of the file:
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@@
 <setting verticaltext="up"/>
 </settings>
-<grid distance="0.05" unitdist="inch" unit="inch" style="lines" multiple="1" display="yes" altdistance="0.005" altunitdist="inch" altunit="inch"/>
+<grid distance="1" unitdist="mm" unit="mm" style="lines" multiple="1" display="yes" altdistance="0.005" altunitdist="inch" altunit="inch"/>
 <layers>
 <layer number="1" name="Top" color="4" fill="1" visible="yes" active="yes"/>
@@
 <layer number="23" name="tOrigins" color="15" fill="1" visible="yes" active="yes"/>
 <layer number="24" name="bOrigins" color="15" fill="1" visible="yes" active="yes"/>
-<layer number="25" name="tNames" color="7" fill="1" visible="no" active="yes"/>
-<layer number="26" name="bNames" color="7" fill="1" visible="no" active="yes"/>
-<layer number="27" name="tValues" color="7" fill="1" visible="no" active="yes"/>
-<layer number="28" name="bValues" color="7" fill="1" visible="no" active="yes"/>
-<layer number="29" name="tStop" color="2" fill="3" visible="no" active="yes"/>
-<layer number="30" name="bStop" color="5" fill="6" visible="no" active="yes"/>
+<layer number="25" name="tNames" color="7" fill="1" visible="yes" active="yes"/>
+<layer number="26" name="bNames" color="7" fill="1" visible="yes" active="yes"/>
+<layer number="27" name="tValues" color="7" fill="1" visible="yes" active="yes"/>
+<layer number="28" name="bValues" color="7" fill="1" visible="yes" active="yes"/>
+<layer number="29" name="tStop" color="2" fill="3" visible="yes" active="yes"/>
+<layer number="30" name="bStop" color="5" fill="6" visible="yes" active="yes"/>
 <layer number="31" name="tCream" color="7" fill="4" visible="yes" active="yes"/>
-<layer number="32" name="bCream" color="7" fill="5" visible="no" active="yes"/>
-<layer number="33" name="tFinish" color="6" fill="3" visible="no" active="yes"/>
-<layer number="34" name="bFinish" color="6" fill="6" visible="no" active="yes"/>
-<layer number="35" name="tGlue" color="7" fill="4" visible="no" active="yes"/>
-<layer number="36" name="bGlue" color="7" fill="5" visible="no" active="yes"/>
-<layer number="37" name="tTest" color="7" fill="1" visible="no" active="yes"/>
-<layer number="38" name="bTest" color="7" fill="1" visible="no" active="yes"/>
-<layer number="39" name="tKeepout" color="4" fill="11" visible="no" active="yes"/>
-<layer number="40" name="bKeepout" color="1" fill="11" visible="no" active="yes"/>
-<layer number="41" name="tRestrict" color="4" fill="10" visible="no" active="yes"/>
-<layer number="42" name="bRestrict" color="1" fill="10" visible="no" active="yes"/>
-<layer number="43" name="vRestrict" color="2" fill="10" visible="no" active="yes"/>
-<layer number="44" name="Drills" color="7" fill="1" visible="no" active="yes"/>
+<layer number="32" name="bCream" color="7" fill="5" visible="yes" active="yes"/>
+<layer number="33" name="tFinish" color="6" fill="3" visible="yes" active="yes"/>
+<layer number="34" name="bFinish" color="6" fill="6" visible="yes" active="yes"/>
+<layer number="35" name="tGlue" color="7" fill="4" visible="yes" active="yes"/>
+<layer number="36" name="bGlue" color="7" fill="5" visible="yes" active="yes"/>
+<layer number="37" name="tTest" color="7" fill="1" visible="yes" active="yes"/>
+<layer number="38" name="bTest" color="7" fill="1" visible="yes" active="yes"/>
+<layer number="39" name="tKeepout" color="4" fill="11" visible="yes" active="yes"/>
+<layer number="40" name="bKeepout" color="1" fill="11" visible="yes" active="yes"/>
+<layer number="41" name="tRestrict" color="4" fill="10" visible="yes" active="yes"/>
+<layer number="42" name="bRestrict" color="1" fill="10" visible="yes" active="yes"/>
+<layer number="43" name="vRestrict" color="2" fill="10" visible="yes" active="yes"/>
+<layer number="44" name="Drills" color="7" fill="1" visible="yes" active="yes"/>
 <layer number="45" name="Holes" color="7" fill="1" visible="yes" active="yes"/>
-<layer number="46" name="Milling" color="3" fill="1" visible="no" active="yes"/>
+<layer number="46" name="Milling" color="3" fill="1" visible="yes" active="yes"/>
 <layer number="47" name="Measures" color="7" fill="1" visible="yes" active="yes"/>
-<layer number="48" name="Document" color="7" fill="1" visible="no" active="yes"/>
+<layer number="48" name="Document" color="7" fill="1" visible="yes" active="yes"/>
 <layer number="49" name="ReferenceLC" color="13" fill="1" visible="yes" active="yes"/>
-<layer number="50" name="ReferenceLS" color="12" fill="1" visible="no" active="yes"/>
+<layer number="50" name="ReferenceLS" color="12" fill="1" visible="yes" active="yes"/>
 <layer number="51" name="tDocu" color="6" fill="1" visible="yes" active="yes"/>
-<layer number="52" name="bDocu" color="7" fill="1" visible="no" active="yes"/>
+<layer number="52" name="bDocu" color="7" fill="1" visible="yes" active="yes"/>
 <layer number="91" name="Nets" color="2" fill="1" visible="no" active="no"/>
 <layer number="92" name="Busses" color="1" fill="1" visible="no" active="no"/>
@@
 <layer number="115" name="ReferenceISLANDS" color="7" fill="1" visible="no" active="no"/>
 <layer number="116" name="Patch_BOT" color="7" fill="1" visible="no" active="no"/>
-<layer number="117" name="PM_Ref" color="26" fill="1" visible="no" active="yes"/>
+<layer number="117" name="PM_Ref" color="26" fill="1" visible="yes" active="yes"/>
 <layer number="118" name="Rect_Pads" color="7" fill="1" visible="no" active="no"/>
-<layer number="119" name="PF_Ref" color="31" fill="1" visible="no" active="yes"/>
-<layer number="120" name="WFL_Ref" color="25" fill="1" visible="no" active="yes"/>
+<layer number="119" name="PF_Ref" color="31" fill="1" visible="yes" active="yes"/>
+<layer number="120" name="WFL_Ref" color="25" fill="1" visible="yes" active="yes"/>
 <layer number="121" name="_tsilk" color="7" fill="1" visible="no" active="no"/>
 <layer number="122" name="_bsilk" color="7" fill="1" visible="no" active="no"/>
@@
 <element name="U$42" library="buzzard_labels (6)" package="_#PWM30" value="" x="43.688" y="42.164" smashed="yes" rot="R90"/>
 <element name="U$43" library="buzzard_labels (6)" package="NC7" value="" x="23.876" y="44.958" smashed="yes" rot="R90"/>
-<element name="U$44" library="Redfive_logo#05#png (1)" package="REDFIVE_LOGO#05#PNG" value="" x="53.975" y="21.59" smashed="yes" rot="R90"/>
 <element name="U$45" library="buzzard_labels (7)" package="133" value="" x="24.892" y="35.941" smashed="yes" rot="R90"/>
 <element name="U$46" library="buzzard_labels (7)" package="PWR0" value="" x="24.892" y="23.495" smashed="yes" rot="R90"/>
@@
 <element name="TP4" library="SparkFun-Connectors" package="PAD.03X.03" value="TEST-POINT3" x="43.18" y="16.51" smashed="yes" rot="MR0"/>
 <element name="TP5" library="SparkFun-Connectors" package="PAD.03X.03" value="TEST-POINT3" x="30.48" y="13.97" smashed="yes" rot="MR0"/>
+<element name="U$52" library="Redfive_logo#05#png (2)" package="REDFIVE_LOGO#05#PNG" value="" x="54" y="22" rot="R90"/>
 </elements>
 <signals>

Commit message: Adding prod_id to JTAG
Parts:
- J5: value CORTEX_JTAG_DEBUG_SMD -> JTAG
Changed lines of the file:
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@@
 <element name="F1" library="SparkFun-Fuses" package="0805" value="6V 0.5A" x="6.35" y="29.845" smashed="yes">
 <attribute name="NAME" x="6.35" y="30.734" size="0.6096" layer="25" font="vector" ratio="20" align="bottom-center"/>
-<attribute name="PROD_ID" value="13945" x="6.35" y="29.845" size="1.778" layer="27" display="off"/>
+<attribute name="PROD_ID" value="RES-13945" x="6.35" y="29.845" size="1.778" layer="27" display="off"/>
 <attribute name="VALUE" x="6.35" y="28.956" size="0.6096" layer="27" font="vector" ratio="20" align="top-center"/>
 </element>
@@
 <attribute name="PROD_ID" value="IC-14494" x="41.91" y="34.29" size="1.778" layer="27" display="off"/>
 </element>
-<element name="J5" library="SparkFun-Connectors" package="2X5-SMD-1.27MM" value="CORTEX_JTAG_DEBUG_SMD" x="43.18" y="17.78" smashed="yes" rot="R180"/>
+<element name="J5" library="SparkFun-Connectors" package="2X5-SMD-1.27MM" value="JTAG" x="43.18" y="17.78" smashed="yes" rot="R180">
+<attribute name="PROD_ID" value="CONN-14503" x="43.18" y="17.78" size="1.778" layer="27" rot="R180" display="off"/>
+<attribute name="VALUE" value="JTAG" x="43.18" y="17.78" size="1.778" layer="27" rot="R180" display="off"/>
+</element>
 <element name="C1" library="SparkFun-Capacitors" package="0603" value="10uF" x="49.53" y="38.354" smashed="yes">
 <attribute name="NAME" x="49.53" y="39.116" size="0.6096" layer="25" font="vector" ratio="20" align="bottom-center"/>

Commit message: v02
Parts:
- removed D3: YELLOW, SparkFun-LED:LED-1206-HIDDENSILK
- removed LED5: GREEN, SparkFun-LED:LED-1206
- removed R11, R13, R17: 22, SparkFun-Resistors:0603
- removed R12, R16: 4.7k, SparkFun-Resistors:0603
- removed U1: CH340C, SparkFun-IC-Comms:SO016
- added C27, C28, C29: 0.1uF, SparkFun-Capacitors:0603
- added C30: 10uF, SparkFun-Capacitors:0603
- added D5: YELLOW, SparkFun-LED:LED-1206-HIDDENSILK
- added J1: AVR_SPI_PROG_3X2PTH, SparkFun-Connectors:2X3
- added LED3: GREEN, SparkFun-LED:LED-1206
- added R20: 100k, SparkFun-Resistors:0603
- added R21, R22: 4.7k, SparkFun-Resistors:0603
- added TP6, TP7, TP8: TEST-POINT3, SparkFun-Connectors:PAD.03X.03
- added U$44: MK22FN128VLH10, SparkFun-IC-Comms:LQFP-64
- C17: value 10nF -> 0.1uF
- moved LOGO1 34.5 mm to (57.7, 32.9)
- moved R3 31.8 mm to (29.2, 41.3), turned to 180 degrees
- moved R5 25.5 mm to (29.2, 43.2)
- moved U5 19.0 mm to (38.1, 40.6), turned to 0 degrees
- moved R8 16.0 mm to (36.2, 34.3), turned to 0 degrees
- moved C26 13.9 mm to (36.2, 32.4)
- moved C25 13.8 mm to (36.2, 30.5)
- moved R7 11.6 mm to (56.8, 24.1), turned to 270 degrees
- moved Y2 9.53 mm to (40.0, 31.4), turned to 135 degrees
- moved D2 9.18 mm to (58.7, 24.1), turned to 90 degrees
- moved C11 8.76 mm to (41.9, 22.9), turned to 0 degrees
- moved C13 8.68 mm to (36.2, 24.8)
- moved C7 8.68 mm to (36.2, 21.0)
- moved C6 8.68 mm to (36.2, 22.9)
- moved C8 8.68 mm to (36.2, 19.1)
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Connections:
- removed net N$11: JP2.7A, JP2.7B, R11.2
- removed net N$14: J2.A6, J2.B6, U1.5
- removed net N$16: JP2.5A, JP2.5B, R17.2
- removed net N$4: JP2.6A, JP2.6B, R13.2
- removed net N$5: LED5.A, R16.1
- removed net N$9: D3.A, R12.1
- new net D+: J2.A6, J2.B6, U$44.5
- new net D-: J2.A7, J2.B7, U$44.6
- new net DBG_RESET: J1.4, R20.1, TP8.P$1, U$44.34
- new net DBG_SWDCLK: J1.3, U$44.22
- new net DBG_SWDIO: J1.1, U$44.25
- new net DBG_SWO: J1.5, U$44.24
- net !RESET: now also U$44.64; no longer U1.13
- net 3.3V: now also C17.1, C18.1, C27.1, C28.1, C29.1, C30.1, J1.2, R20.2, R21.2, R22.2, TP6.P$1, U$44.13, U$44.14, U$44.21, U$44.26, U$44.3, U$44.30, U$44.48, U$44.7
- net 5V: no longer C18.1, R12.2, R16.2, U1.16
- net GND: now also C27.2, C28.2, C29.2, C30.2, J1.6, TP7.P$1, U$44.15, U$44.16, U$44.31, U$44.4, U$44.47; no longer U1.1
- net N$13: now also D5.A, R21.1; no longer J2.A7, J2.B7, U1.6
- net N$6: now also LED3.A, R22.1; no longer C17.1, U1.4
- net RXI: now also D5.C, U$44.39; no longer D3.C, U1.2
- net SPI_MISO: now also JP2.6A, JP2.6B; no longer R13.1
- net SPI_MOSI: now also JP2.7A, JP2.7B; no longer R11.1
- net SPI_SCK: now also JP2.5A, JP2.5B; no longer R17.1
- net TCK: now also U$44.62
- net TDI: now also U$44.59
- net TDO: now also U$44.2
- net TMS: now also U$44.63
- net TXO: now also LED3.C, U$44.40; no longer LED5.C, U1.3
Routing:
- net 3.3V: track 193.0 -> 263.0 mm, vias 10 -> 19
- net TDI: track 17.6 -> 62.6 mm, vias 1 -> 2
- net TDO: track 13.1 -> 57.8 mm
- net TMS: track 16.0 -> 52.6 mm
- net TCK: track 19.4 -> 52.9 mm, vias 3 -> 2
- net SPI_SCK: track 29.0 -> 55.5 mm, vias 2 -> 4
- net SPI_MOSI: track 11.5 -> 37.0 mm
- net SPI_MISO: track 13.3 -> 38.0 mm
- net IO11: track 62.9 -> 38.4 mm, vias 2 -> 0
- net DBG_RESET: track 0.00 -> 22.4 mm, vias 0 -> 1
- net 5V: track 101.1 -> 78.9 mm, vias 26 -> 23
- net DBG_SWO: track 0.00 -> 19.8 mm, vias 0 -> 1
- net IO9: track 53.3 -> 35.7 mm, vias 2 -> 0
- net IO10: track 58.1 -> 40.4 mm, vias 2 -> 0
- net DBG_SWDCLK: track 0.00 -> 17.6 mm, vias 0 -> 1
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
Commit message: pre design review number 2
Routing:
- net 3.3V: track 263.0 -> 261.6 mm
Other:
- board text added: "v02"
- board text removed: "v01"
Changed lines of the file:
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@@
 <wire x1="66.04" y1="51.816" x2="66.04" y2="40.386" width="0.2032" layer="20"/>
 <text x="0" y="-0.0635" size="0.0254" layer="214" font="vector">D:/SmartProjects/Snc/a4_bn_logo2.bmp</text>
-<text x="6.81" y="0.508" size="1.27" layer="16" font="vector" ratio="20" rot="MR0">v01</text>
+<text x="6.81" y="0.508" size="1.27" layer="16" font="vector" ratio="20" rot="MR0">v02</text>
 <text x="31" y="-17" size="1.778" layer="51" font="vector">A. England</text>
 <rectangle x1="0.635" y1="22.352" x2="2.032" y2="30.607" layer="43"/>
@@
 <element name="TP7" library="SparkFun-Connectors" package="PAD.03X.03" value="TEST-POINT3" x="40.64" y="3.81" rot="MR0"/>
 <element name="U$44" library="SparkFun-IC-Comms" package="LQFP-64" value="MK22FN128VLH10" x="18" y="34">
-<attribute name="PROD_ID" value="" x="18" y="34" size="1.778" layer="27" display="off"/>
+<attribute name="PROD_ID" value="IC-14611" x="18" y="34" size="1.778" layer="27" display="off"/>
 <attribute name="VALUE" value="MK22FN128VLH10" x="18" y="34" size="1.778" layer="27" display="off"/>
 </element>
@@
 <wire x1="12.692" y1="28.694" x2="13.208" y2="29.21" width="0.2032" layer="1"/>
 <wire x1="13.208" y1="29.21" x2="16.25" y2="29.21" width="0.2032" layer="1"/>
-<wire x1="20.75" y1="28.2" x2="20.75" y2="27.94" width="0.2032" layer="1"/>
-<wire x1="20.75" y1="26.455" x2="20.955" y2="26.25" width="0.2032" layer="1"/>
 <wire x1="20.75" y1="28.2" x2="20.75" y2="28.526" width="0.2032" layer="1"/>
 <wire x1="18.917" y1="30.359" x2="18.796" y2="30.359" width="0.2032" layer="1"/>
@@
 <wire x1="46.14" y1="27.266" x2="46.14" y2="26.67" width="0.2032" layer="1"/>
 <wire x1="45.92" y1="27.486" x2="46.14" y2="27.266" width="0.2032" layer="1"/>
-<wire x1="46.14" y1="26.67" x2="46.14" y2="26.25" width="0.2032" layer="1"/>
 <wire x1="41.06" y1="29.63" x2="41.06" y2="26.67" width="0.2032" layer="1"/>
 <wire x1="42.164" y1="32.131" x2="42.164" y2="30.734" width="0.2032" layer="1"/>
@@
 <wire x1="47.83436875" y1="29.337" x2="48.46936875" y2="29.972" width="0.2032" layer="1"/>
 <wire x1="56.769" y1="23.28" x2="56.769" y2="19.73" width="0.2032" layer="1"/>
-<wire x1="48.71556875" y1="23.15373125" x2="48.68073125" y2="23.15373125" width="0.2032" layer="1"/>
 <via x="48.68073125" y="23.15373125" extent="1-16" drill="0.35"/>
 <via x="46.736" y="23.495" extent="1-16" drill="0.35"/>
@@
 <wire x1="44.227" y1="38.6052" x2="44.2242" y2="38.608" width="0.2032" layer="16"/>
 <wire x1="48.4692625" y1="38.6052" x2="44.227" y2="38.6052" width="0.2032" layer="16"/>
-<wire x1="52.705" y1="33.87" x2="52.236" y2="33.87" width="0.2032" layer="1"/>
 <via x="50.038" y="34.671" extent="1-16" drill="0.35"/>
 <wire x1="48.645" y1="34.89" x2="49.819" y2="34.89" width="0.2032" layer="1"/>
@@
 <wire x1="29.21" y1="16.002" x2="29.21" y2="11.43" width="0.2032" layer="1"/>
 <via x="48.26" y="23.749" extent="1-16" drill="0.35"/>
-<wire x1="45.2595375" y1="25.7466625" x2="45.1908625" y2="25.7466625" width="0.1524" layer="16"/>
 <wire x1="43.942" y1="24.4978" x2="45.1908625" y2="25.7466625" width="0.2032" layer="16"/>
 <wire x1="45.9872" y1="25.7678" x2="48.006" y2="23.749" width="0.2032" layer="16"/>
@@
 <wire x1="48.645" y1="35.69" x2="52.77894375" y2="35.69" width="0.2032" layer="1"/>
 <wire x1="52.77894375" y1="35.69" x2="54.140471875" y2="34.328471875" width="0.2032" layer="1"/>
-<wire x1="55.88" y1="0.8636" x2="56.0483375" y2="0.8636" width="0.2032" layer="1"/>
 <wire x1="54.140471875" y1="8.089528125" x2="55.88" y2="6.35" width="0.2032" layer="1"/>
 <wire x1="55.88" y1="6.35" x2="55.88" y2="0.8636" width="0.2032" layer="1"/>

Commit message: small schematic tweaks, thanks pete for notes
Parts:
- J1: value AVR_SPI_PROG_3X2PTH -> FEMALE 2x3
Changed lines of the file:
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@@
 <attribute name="PROD_ID" value="CAP-00810" x="20.955" y="25.4" size="1.778" layer="27" rot="R270" display="off"/>
 </element>
-<element name="J1" library="SparkFun-Connectors" package="2X3" value="AVR_SPI_PROG_3X2PTH" x="24.96" y="19.57" rot="R270"/>
+<element name="J1" library="SparkFun-Connectors" package="2X3" value="FEMALE 2x3" x="24.96" y="19.57" rot="R270">
+<attribute name="PROD_ID" value="CONN-11566" x="24.96" y="19.57" size="1.778" layer="27" rot="R270" display="off"/>
+<attribute name="VALUE" value="FEMALE 2x3" x="24.96" y="19.57" size="1.778" layer="27" rot="R270" display="off"/>
+</element>
 <element name="TP8" library="SparkFun-Connectors" package="PAD.03X.03" value="TEST-POINT3" x="27.94" y="21.59" rot="MR0"/>
 <element name="R20" library="SparkFun-Resistors" package="0603" value="100k" x="30.48" y="20.32" rot="R270">
