File: Hardware/RedFive.brd (EAGLE design)
At the start: 68.6 x 53.3 mm, 131 parts, among them IC3 LM1117, J1 FEMALE 2x3, J2 USB Female Type C Connector, J3 POWER_JACKSUPER_BOMB_DIGITY, J4 QWIIC_RIGHT_ANGLE, J5 CORTEX_JTAG_DEBUG_PTH_NS, Q1 1.1A/60V/600mΩ, U2 1.8V, U3 AP2112-3.3V, U4 FE310, U5 32MBit, Y1 32.768KHZ, Y2 16MHz

Commit message: post review changes-v10
Parts:
- removed J1: FEMALE 2x3, SparkFun-Connectors:2X3_POGO
- removed U$51: (no value), Redfive_logo#07#png (1):REDFIVE_LOGO#07#PNG
- added I2C: JUMPER-SMT_3_NO_NO-SILK, SparkFun-Jumpers:SMT-JUMPER_3_NO_NO-SILK
- added TP1, TP2, TP3, TP4, TP5, TP6: TEST-POINT3X5, SparkFun-Connectors:PAD.03X.05
- added U$8: (no value), seggerlogo#png:SEGGERLOGO#PNG
- D5: value YELLOW -> GREEN; device SparkFun-LED:LED-1206-HIDDENSILK -> SparkFun-LED:LED-1206
- J4: value QWIIC_RIGHT_ANGLE -> QWIIC
- LED1: value Blue -> BLUE; device SparkFun-LED:LED-1206-HIDDENSILK -> SparkFun-LED:LED-1206
- LED3: value GREEN -> Yellow
- moved LOGO1 23.3 mm to (42.0, 15.6)
- moved U$52 1.61 mm to (52.7, 15.7)
- moved D1 1.42 mm to (15.9, 8.26)
- moved JP3 1.27 mm to (15.2, 2.54)
- moved R2 0.06 mm to (29.2, 24.0)
- renumbered U$44 to U6
Connections:
- new net N$4: I2C.3, R10.2
- new net N$5: I2C.1, R9.2
- net 3.3V: now also I2C.2, TP1.P$1; no longer J1.P$2, R10.2, R9.2
- net DBG_RESET: now also TP2.P$1; no longer J1.P$4
- net DBG_SWDCLK: now also TP5.P$1; no longer J1.P$3
- net DBG_SWDIO: now also TP4.P$1; no longer J1.P$1
- net DBG_SWO: now also TP6.P$1; no longer J1.P$5
- net GND: now also TP3.P$1; no longer J1.P$6
Routing:
- net 3.3V: track 260.7 -> 254.0 mm, vias 20 -> 19
- net QSPI_SCK: track 11.9 -> 8.73 mm
- net N$5: track 0.00 -> 1.65 mm
- net N$4: track 0.00 -> 1.59 mm
- net PWRIN: track 15.8 -> 17.3 mm
- net QSPI_3: track 19.6 -> 18.2 mm
- net TDO: track 61.2 -> 60.2 mm
- net QSPI_CS: track 16.4 -> 17.2 mm
- net SDA: track 90.7 -> 91.4 mm
- net VIN: track 62.2 -> 61.5 mm
- net DBG_SWDIO: track 14.4 -> 15.1 mm
- net DBG_SWDCLK: track 17.6 -> 18.2 mm
- net DBG_SWO: track 19.8 -> 20.4 mm
- net !RESET: vias 4 -> 6
- net GND: vias 73 -> 101
Other:
- board text added: "v10"
- board text removed: "v02"

Commit message: post checklist changes
Parts:
- added U$11: (no value), buzzard_labels:I2C0
- U2: value 1.8V -> AP2127K-1.8V
Changed lines of the file:
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@@
 <element name="JP15" library="SparkFun" package="FIDUCIAL-1X2" value="FIDUCIAL1X2" x="3.81" y="45.72" smashed="yes" rot="MR0"/>
 <element name="JP16" library="SparkFun" package="FIDUCIAL-1X2" value="FIDUCIAL1X2" x="66.04" y="11.43" smashed="yes" rot="MR0"/>
-<element name="U2" library="SparkFun-IC-Power" package="SOT23-5" value="1.8V" x="15.24" y="24.4" smashed="yes">
+<element name="U2" library="SparkFun-IC-Power" package="SOT23-5" value="AP2127K-1.8V" x="15.24" y="24.4" smashed="yes">
 <attribute name="NAME" x="14.351" y="26.559" size="0.4064" layer="25"/>
 <attribute name="PROD_ID" value="VREG-14239" x="15.24" y="24.4" size="1.778" layer="27" display="off"/>
-<attribute name="VALUE" x="14.2875" y="24.2095" size="0.4064" layer="27"/>
+<attribute name="VALUE" value="AP2127K-1.8V" x="14.2875" y="24.2095" size="0.4064" layer="27"/>
 </element>
 <element name="C9" library="SparkFun-Capacitors" package="0603" value="1.0uF" x="36.195" y="28.575" smashed="yes" rot="R180">
@@
 <element name="TP6" library="SparkFun-Connectors" package="PAD.03X.05" value="TEST-POINT3X5" x="25.4" y="13.97" rot="MR0"/>
 <element name="U$8" library="seggerlogo#png" package="SEGGERLOGO#PNG" value="" x="62.23" y="26.67" rot="MR0"/>
+<element name="U$11" library="buzzard_labels" package="I2C0" value="" x="56.769" y="20.701"/>
 </elements>
 <signals>

Commit message: updating R8 to 100 Ohm
Parts:
- R8: value 100k -> 100
Changed lines of the file:
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@@
 <attribute name="VALUE" x="36.195" y="31.623" size="0.6096" layer="27" font="vector" ratio="20" align="top-center"/>
 </element>
-<element name="R8" library="SparkFun-Resistors" package="0603" value="100k" x="36.195" y="34.29" smashed="yes">
+<element name="R8" library="SparkFun-Resistors" package="0603" value="100" x="36.195" y="34.29" smashed="yes">
 <attribute name="NAME" x="36.195" y="35.052" size="0.6096" layer="25" font="vector" ratio="20" align="bottom-center"/>
-<attribute name="PROD_ID" value="RES-07828" x="36.195" y="34.29" size="1.778" layer="27" display="off"/>
-<attribute name="VALUE" x="36.195" y="33.528" size="0.6096" layer="27" font="vector" ratio="20" align="top-center"/>
+<attribute name="PROD_ID" value="RES-07863" x="36.195" y="34.29" size="1.778" layer="27" display="off"/>
+<attribute name="VALUE" value="100" x="36.195" y="33.528" size="0.6096" layer="27" font="vector" ratio="20" align="top-center"/>
 </element>
 <element name="R9" library="SparkFun-Resistors" package="0603" value="4.7k" x="57.785" y="16.51" smashed="yes" rot="R90">
@@
 <element name="D5" library="SparkFun-LED" package="LED-1206" value="GREEN" x="29.21" y="29.972" smashed="yes">
 <attribute name="NAME" x="29.21" y="30.9245" size="0.6096" layer="25" font="vector" ratio="20" align="bottom-center"/>
-<attribute name="PROD_ID" value="DIO-00862" x="29.21" y="33.972" size="1.778" layer="27" display="off"/>
+<attribute name="PROD_ID" value="DIO-09910" x="29.21" y="33.972" size="1.778" layer="27" display="off"/>
 <attribute name="VALUE" value="GREEN" x="29.21" y="29.0195" size="0.6096" layer="27" font="vector" ratio="20" align="top-center"/>
 </element>
